Commit message: fix sim to work state

File: src/t21_sim/config/t21.ros2_control.xacro (robot description, xacro)
@@ -13,5 +13,5 @@
       </hardware>
       <!-- виртуальный сустав линейной скорости -->
-      <joint name="wheel_left_joint">
+      <joint name="left_wheel_joint">
         <command_interface name="velocity"/>
         <state_interface   name="velocity"/>
@@ -19,14 +19,14 @@
       </joint>
       <!-- виртуальный сустав угловой скорости -->
-      <joint name="wheel_right_joint">
+      <joint name="right_wheel_joint">
         <command_interface name="velocity"/>
         <state_interface   name="velocity"/>
         <state_interface name="position"/>
       </joint>
-      <!-- реальный сустав флиппера / стрелы -->
-      <!--joint name="${prefix}geom_joint">
+      <!--реальный сустав флиппера / стрелы -->
+      <joint name="fliper_joint">
         <command_interface name="position"/>
         <state_interface   name="position"/>
-      </joint-->
+      </joint>
     </ros2_control>
     <gazebo>

File: src/t21_sim/urdf/tracked_robot.urdf.xacro (robot description, xacro)
@@ -1,174 +1,175 @@
 <?xml version="1.0"?>
-<robot name="t21" xmlns:xacro="http://www.ros.org/wiki/xacro">
-  <!-- ──────────────── CONSTANTS ──────────────── -->
-  <xacro:property name="scale_small" value="1"/>
-  <xacro:property name="scale_big" value="0.001"/>
-  <xacro:property name="color_grey" value="0.6 0.6 0.6 1.0"/>
-  <xacro:property name="wheel_radius" value="0.05"/>
-  <xacro:property name="wheel_length" value="0.02"/>
-  <xacro:property name="lidar_radius" value="0.03"/>
-  <xacro:property name="lidar_length" value="0.05"/>
-  <!-- ──────────────── MACROS ──────────────── -->
-  <xacro:macro name="cylinder_link" params="name radius length mass *visual *collision">
-    <link name="${name}">
-      <inertial>
-        <mass value="${mass}"/>
-        <origin xyz="0 0 0" rpy="0 0 0"/>
-        <inertia ixx="${mass*(3*radius*radius + length*length)/12}" ixy="0" ixz="0"
-                 iyy="${mass*(3*radius*radius + length*length)/12}" iyz="0"
-                 izz="${mass*(radius*radius)/2}"/>
-      </inertial>
-      <visual>
-        <origin xyz="0 0 0" rpy="0 0 0"/>
+<robot xmlns:xacro="http://www.ros.org/wiki/xacro" name="tracked_robot">
+  <!-- Materials -->
+  <material name="grey">
+    <color rgba="0.56471 0.56471 0.56471 1"/>
+  </material>
+  <material name="white">
+    <color rgba="1 1 1 0"/>
+  </material>
+  <material name="light_blue">
+    <color rgba="0.79216 0.81961 0.93333 1"/>
+  </material>
+  <!-- Base Link -->
+  <link name="base_link">
+    <inertial>
+      <origin xyz="-0.0023851 -2.6804E-12 0.049804" rpy="0 0 0"/>
+      <mass value="24.218"/>
+      <inertia ixx="0.38879" ixy="-2.3825E-10" ixz="-0.0015299" iyy="0.63474" iyz="-6.2968E-13" izz="0.97264"/>
+    </inertial>
+    <visual>
+      <origin xyz="0 0 0" rpy="0 0 0"/>
+      <geometry>
+        <mesh filename="file://$(find t21_sim)/meshes/base_link.STL"/>
+      </geometry>
+      <material name="grey"/>
+    </visual>
+    <collision>
+      <origin xyz="0 0 0" rpy="0 0 0"/>
+      <geometry>
+        <mesh filename="file://$(find t21_sim)/meshes/base_link.STL"/>
+      </geometry>
+    </collision>
+  </link>
+  <!-- Left Wheel -->
+  <link name="left_wheel_link">
+    <inertial>
+      <origin xyz="0 -0.015 0" rpy="0 0 0"/>
+      <mass value="0.50915"/>
+      <inertia ixx="0.00072583" ixy="3.5474E-36" ixz="-1.9259E-34" iyy="0.0013753" iyz="-2.0195E-21" izz="0.00072583"/>
+    </inertial>
+    <visual>
+      <origin xyz="0 0 0" rpy="0 0 0"/>
+      <geometry>
+        <mesh filename="file://$(find t21_sim)/meshes/left_wheel_link.STL" scale="1.0 0.1 1.0"/>
+      </geometry>
+      <material name="white"/>
+    </visual>
+    <collision>
+      <origin xyz="0 0 0" rpy="0 0 0"/>
+      <geometry>
+        <mesh filename="file://$(find t21_sim)/meshes/left_wheel_link.STL" scale="1.0 0.1 1.0"/>
+      </geometry>
+    </collision>
+  </link>
+  <joint name="left_wheel_joint" type="continuous">
+    <origin xyz="-0.015028 0.2025 0.04" rpy="0 0 0"/>
+    <parent link="base_link"/>
+    <child link="left_wheel_link"/>
+    <axis xyz="0 1 0"/>
+    <limit effort="10" velocity="10"/>
+    <dynamics friction="0.1"/>
+  </joint>
+  <!-- Right Wheel -->
+  <link name="right_wheel_link">
+    <inertial>
+      <origin xyz="0 0.015 0" rpy="0 0 0"/>
+      <mass value="0.50915"/>
+      <inertia ixx="0.00072583" ixy="-2.0887E-36" ixz="9.1015E-36" iyy="0.0013753" iyz="4.7568E-21" izz="0.00072583"/>
+    </inertial>
+    <visual>
+      <origin xyz="0 0 0" rpy="0 0 0"/>
+      <geometry>
+        <mesh filename="file://$(find t21_sim)/meshes/right_wheel_link.STL" scale="1.0 0.1 1.0"/>
+      </geometry>
+      <material name="white"/>
+    </visual>
+    <collision>
+      <origin xyz="0 0 0" rpy="0 0 0"/>
+      <geometry>
+        <mesh filename="file://$(find t21_sim)/meshes/right_wheel_link.STL" scale="1.0 0.1 1.0"/>
+      </geometry>
+    </collision>
+  </link>
+  <joint name="right_wheel_joint" type="continuous">
+    <origin xyz="-0.015028 -0.2025 0.04" rpy="0 0 0"/>
+    <parent link="base_link"/>
+    <child link="right_wheel_link"/>
+    <axis xyz="0 1 0"/>
+    <limit effort="10" velocity="10"/>
+    <dynamics friction="0.1"/>
+  </joint>
+  <!-- Flipper -->
+  <link name="fliper_link">
+    <inertial>
+      <origin xyz="0.10581 -0.24294 -0.0083667" rpy="0 0 0"/>
+      <mass value="2.7683"/>
+      <inertia ixx="0.0029923" ixy="1.2514E-05" ixz="0.0017391" iyy="0.037286" iyz="-9.2678E-07" izz="0.03494"/>
+    </inertial>
+    <visual>
+      <origin xyz="0 0 0" rpy="0 0 0"/>
+      <geometry>
+        <mesh filename="file://$(find t21_sim)/meshes/fliper_link.STL"/>
+      </geometry>
+      <material name="light_blue"/>
+    </visual>
+    <collision>
+      <origin xyz="0 0 0" rpy="0 0 0"/>
+      <geometry>
+        <mesh filename="file://$(find t21_sim)/meshes/fliper_link.STL"/>
+      </geometry>
+    </collision>
+  </link>
+  <joint name="fliper_joint" type="revolute">
+    <origin xyz="0.222 0.2435 0.04" rpy="0 0 0"/>
+    <parent link="base_link"/>
+    <child link="fliper_link"/>
+    <axis xyz="0 -1 0"/>
+    <limit lower="0" upper="0" effort="10" velocity="10"/>
+  </joint>
+  <link name="big_box_link">
+      <collision>
+        <origin rpy="0 0 0" xyz="0 0 0"/>
         <geometry>
-          <cylinder radius="${radius}" length="${length}"/>
-        </geometry>
-        <xacro:insert_block name="visual"/>
-      </visual>
-      <collision>
-        <origin xyz="0 0 0" rpy="0 0 0"/>
-        <geometry>
-          <cylinder radius="${radius}" length="${length}"/>
-        </geometry>
-        <xacro:insert_block name="collision"/>
-      </collision>
-    </link>
-  </xacro:macro>
-  <!-- Основной макрос для меш-объектов -->
-  <xacro:macro name="add_link" params="name mesh scale color rpy xyz mass">
-    <link name="${name}">
-      <inertial>
-        <mass value="${mass}"/>
-        <origin xyz="0 0 0" rpy="0 0 0"/>
-        <inertia ixx="${mass*0.1}" ixy="0" ixz="0"
-                 iyy="${mass*0.1}" iyz="0"
-                 izz="${mass*0.1}"/>
-      </inertial>
-      <collision>
-        <origin rpy="${rpy}" xyz="${xyz}"/>
-        <geometry>
-          <mesh filename="package://t21_sim/meshes/${mesh}"
-                scale="${scale} ${scale} ${scale}"/>
+          <mesh filename="file://$(find t21_sim)/meshes/big_box.stl"
+                scale="0.001 0.001 0.001"/>
         </geometry>
       </collision>
       <visual>
-        <origin rpy="${rpy}" xyz="${xyz}"/>
+        <origin rpy="0 0 0" xyz="0 0 0"/>
         <geometry>
-          <mesh filename="package://t21_sim/meshes/${mesh}"
-                scale="${scale} ${scale} ${scale}"/>
+          <mesh filename="file://$(find t21_sim)/meshes/big_box.stl"
+                scale="0.001 0.001 0.001"/>
         </geometry>
-        <material name="Grey">
-          <color rgba="${color}"/>
-        </material>
+        <material name="light_blue"/>
       </visual>
-    </link>
-  </xacro:macro>
-  <link name="world"/>
-  <!-- ──────────────── BASE ──────────────── -->
-  <xacro:add_link name="base_link"
-                 mesh="base.stl"
-                 scale="${scale_small}"
-                 color="${color_grey}"
-                 rpy="0 0 0"
-                 xyz="0 0 0"
-                 mass="5.0"/>
-  <joint name="base_joint" type="fixed">
-    <parent link="world"/>
-    <child link="base_link"/>
-    <origin xyz="0 0 0" rpy="0 0 0"/>
+  </link>
+  <joint name="big_box_joint" type="fixed">
+    <parent link="base_link"/><child link="big_box_link"/>
+    <origin xyz="0.265 -0.093 0.1" rpy="0 0 0"/>
   </joint>
-  <!-- ──────────────── FLIPPER / GEOMETRY ──────────────── -->
-  <xacro:add_link name="geom_link"
-                 mesh="fliper.stl"
-                 scale="${scale_small}"
-                 color="${color_grey}"
-                 rpy="0 0 0"
-                 xyz="0 0 0"
-                 mass="1.5"/>
-  <joint name="geom_joint" type="revolute">
-    <parent link="base_link"/>
-    <child link="geom_link"/>
-    <origin xyz="0.22513 0.1925 0.07335" rpy="-1.57 4.71239 0"/>
-    <axis xyz="0 0 1"/>
-    <limit lower="0.174533" upper="5.93412" effort="1000" velocity="1"/>
+  <link name="lidar_link">
+    <inertial><mass value="1e-6"/><origin xyz="0 0 0" rpy="0 0 0"/>
+      <inertia ixx="1e-6" iyy="1e-6" izz="1e-6" ixy="0" ixz="0" iyz="0"/>
+    </inertial>
+  </link>
+  <joint name="lidar_joint" type="fixed">
+    <parent link="big_box_link"/><child link="lidar_link"/>
+    <origin xyz="-0.111 0.092 0.118" rpy="0 0 0"/>
   </joint>
-  <!-- ──────────────── WHEELS ──────────────── -->
-  <xacro:cylinder_link name="wheel_left_link"
-                      radius="${wheel_radius}"
-                      length="${wheel_length}"
-                      mass="0.5">
-    <visual>
-      <material name="Invisible">
-        <color rgba="0 0 0 0"/>
-      </material>
-    </visual>
-    <collision/>
-  </xacro:cylinder_link>
-  <joint name="wheel_left_joint" type="continuous">
-    <parent link="base_link"/>
-    <child link="wheel_left_link"/>
-    <origin xyz="0 0.1865 0.065" rpy="0 0 0"/>
-    <axis xyz="0 1 0"/>
-  </joint>
-  <gazebo reference="wheel_left_link">
-    <mu1 value="1.0"/>
-    <mu2 value="0.1"/>
-    <fdir1 value="0 0 0"/>
-    <maxContacts value="1"/>
-    <material>Gazebo/Invisible</material>
+  <!-- Gazebo extensions -->
+  <gazebo reference="base_link">
+    <mu1>0.2</mu1>
+    <mu2>0.2</mu2>
+    <kp>1000000.0</kp>
+    <kd>100.0</kd>
   </gazebo>
-  <xacro:cylinder_link name="wheel_right_link"
-                      radius="${wheel_radius}"
-                      length="${wheel_length}"
-                      mass="0.5">
-    <visual>
-      <material name="Invisible">
-        <color rgba="0 0 0 0"/>
-      </material>
-    </visual>
-    <collision/>
-  </xacro:cylinder_link>
-  <joint name="wheel_right_joint" type="continuous">
-    <parent link="base_link"/>
-    <child link="wheel_right_link"/>
-    <origin xyz="0 -0.1865 0.065" rpy="0 0 0"/>
-    <axis xyz="0 1 0"/>
-  </joint>
-  <gazebo reference="wheel_right_link">
-    <mu1 value="1.0"/>
-    <mu2 value="0.1"/>
-    <fdir1 value="0 0 0"/>
-    <maxContacts value="1"/>
-    <material>Gazebo/Invisible</material>
+  <gazebo reference="left_wheel_link">
+    <mu1>1.0</mu1>
+    <mu2>1.0</mu2>
+    <kp>1000000.0</kp>
+    <kd>100.0</kd>
   </gazebo>
-  <!-- ──────────────── BOX AND SENSORS ──────────────── -->
-  <xacro:add_link name="big_box_link"
-                 mesh="big_box.stl"
-                 scale="${scale_big}"
-                 color="${color_grey}"
-                 rpy="0 0 0"
-                 xyz="0 0 0"
-                 mass="0.3"/>
-  <joint name="big_box_joint" type="fixed">
-    <parent link="base_link"/>
-    <child link="big_box_link"/>
-    <origin xyz="0.265 -0.093 0.133" rpy="0 0 0"/>
-  </joint>
-  <!-- Лидар в виде вертикального цилиндра -->
-  <xacro:cylinder_link name="lidar_link"
-                      radius="${lidar_radius}"
-                      length="${lidar_length}"
-                      mass="0.1">
-    <visual>
-      <material name="DarkGrey">
-        <color rgba="0.2 0.2 0.2 1.0"/>
-      </material>
-    </visual>
-    <collision/>
-  </xacro:cylinder_link>
-  <joint name="lidar_joint" type="fixed">
-    <parent link="big_box_link"/>
-    <child link="lidar_link"/>
-    <origin xyz="-0.111 0.092 0.118" rpy="0 0 1.5708"/> <!-- Повернут на 90 градусов -->
-  </joint>
+  <gazebo reference="right_wheel_link">
+    <mu1>1.0</mu1>
+    <mu2>1.0</mu2>
+    <kp>1000000.0</kp>
+    <kd>100.0</kd>
+  </gazebo>
+  <gazebo reference="fliper_link">
+    <mu1>0.5</mu1>
+    <mu2>0.5</mu2>
+    <kp>1000000.0</kp>
+    <kd>100.0</kd>
+  </gazebo>
 </robot>
