Commit message: Added lidar nodes to recieve data from VLP-16 - launch&config files; started conditions in bringup_t21.launch to add VLP simulation

File: src/tracked_description/urdf/t21.urdf.xacro (robot description, xacro)
@@ -2,4 +2,5 @@
 <robot xmlns:xacro="http://www.ros.org/wiki/xacro" name="t21">
   <xacro:arg name="prefix" default=""/>
+  <xacro:arg name="use_lidar" default="false"/>
   <!-- геометрия -->
   <xacro:include filename="$(find tracked_description)/urdf/tracked_robot.urdf.xacro"/>
@@ -8,3 +9,25 @@
   <!-- вызываем макрос, передавая имя и префикс -->
   <xacro:t21_ros2_control name="t21" prefix="$(arg prefix)"/>
+  <xacro:if value="${use_lidar}">
+    <xacro:VLP-16 parent="lidar_link"
+                name="velodyne"
+                topic="/velodyne_points"
+                organize_cloud="false"
+                hz="10"
+                lasers="16"
+                samples="400"
+                collision_range="0.3"
+                min_range="0.1"
+                max_range="25.0"
+                min_angle="-${pi/2}"
+                max_angle="${pi/2}"
+                gpu="false">
+                <origin xyz="0 0 0" rpy="0 0 0" />
+    </xacro:VLP-16>
+  </xacro:if>
+  <!-- <xacro:include filename="$(find realsense2_description)/urdf/_d415.urdf.xacro"/>
+  <xacro:sensor_d415 parent="front_camera_link" use_nominal_extrinsics="true">
+    <origin xyz="0 0 0" rpy="0 0 0"/>
+  </xacro:sensor_d415>
+  <xacro:include filename="depth_camera.xacro"/> -->
 </robot>

Commit message: Fix arg in urdf to sim_lidar and min_range decreased to 0.5m

File: src/tracked_description/urdf/t21.urdf.xacro (robot description, xacro)
@@ -1,6 +1,9 @@
 <?xml version="1.0"?>
 <robot xmlns:xacro="http://www.ros.org/wiki/xacro" name="t21">
+  <!-- Объявляем аргументы -->
   <xacro:arg name="prefix" default=""/>
-  <xacro:arg name="use_lidar" default="false"/>
+  <xacro:arg name="sim_lidar" default="false"/>
+  <!-- Создаем свойство на основе аргумента -->
+  <xacro:property name="sim_lidar_flag" value="$(arg sim_lidar)"/>
   <!-- геометрия -->
   <xacro:include filename="$(find tracked_description)/urdf/tracked_robot.urdf.xacro"/>
@@ -9,5 +12,8 @@
   <!-- вызываем макрос, передавая имя и префикс -->
   <xacro:t21_ros2_control name="t21" prefix="$(arg prefix)"/>
-  <xacro:if value="${use_lidar}">
+  <!-- блок симуляции VLP-16-->
+  <xacro:include filename="$(find velodyne_description)/urdf/VLP-16.urdf.xacro"/>
+  <!-- Используем свойство вместо прямого аргумента -->
+  <xacro:if value="${sim_lidar_flag == 'true'}">
     <xacro:VLP-16 parent="lidar_link"
                 name="velodyne"
@@ -17,17 +23,11 @@
                 lasers="16"
                 samples="400"
-                collision_range="0.3"
                 min_range="0.1"
                 max_range="25.0"
-                min_angle="-${pi/2}"
-                max_angle="${pi/2}"
+                min_angle="-1.5708"
+                max_angle="1.5708"
                 gpu="false">
-                <origin xyz="0 0 0" rpy="0 0 0" />
+      <origin xyz="0 0 0" rpy="0 0 0" />
     </xacro:VLP-16>
   </xacro:if>
-  <!-- <xacro:include filename="$(find realsense2_description)/urdf/_d415.urdf.xacro"/>
-  <xacro:sensor_d415 parent="front_camera_link" use_nominal_extrinsics="true">
-    <origin xyz="0 0 0" rpy="0 0 0"/>
-  </xacro:sensor_d415>
-  <xacro:include filename="depth_camera.xacro"/> -->
 </robot>

Commit message: add D435 description - by choise; TODO - add param to launch

File: src/tracked_description/urdf/t21.urdf.xacro (robot description, xacro)
@@ -1,9 +1,9 @@
 <?xml version="1.0"?>
-<robot xmlns:xacro="http://www.ros.org/wiki/xacro" name="t21">
+<robot name="t21" xmlns:xacro="http://ros.org/wiki/xacro">
   <!-- Объявляем аргументы -->
   <xacro:arg name="prefix" default=""/>
+  <!-- Использовать симуляцию лидара\камеры -->
   <xacro:arg name="sim_lidar" default="false"/>
-  <!-- Создаем свойство на основе аргумента -->
-  <xacro:property name="sim_lidar_flag" value="$(arg sim_lidar)"/>
+  <xacro:arg name="sim_cam" default="true"/>
   <!-- геометрия -->
   <xacro:include filename="$(find tracked_description)/urdf/tracked_robot.urdf.xacro"/>
@@ -12,8 +12,8 @@
   <!-- вызываем макрос, передавая имя и префикс -->
   <xacro:t21_ros2_control name="t21" prefix="$(arg prefix)"/>
-  <!-- блок симуляции VLP-16-->
-  <xacro:include filename="$(find velodyne_description)/urdf/VLP-16.urdf.xacro"/>
   <!-- Используем свойство вместо прямого аргумента -->
-  <xacro:if value="${sim_lidar_flag == 'true'}">
+  <xacro:if value="${'$(arg sim_lidar)' == 'true'}">
+    <!-- блок симуляции VLP-16-->
+    <xacro:include filename="$(find velodyne_description)/urdf/VLP-16.urdf.xacro"/>
     <xacro:VLP-16 parent="lidar_link"
                 name="velodyne"
@@ -31,3 +31,13 @@
     </xacro:VLP-16>
   </xacro:if>
+  <xacro:if value="${'$(arg sim_cam)' == 'true'}">
+    <xacro:include filename="$(find realsense2_description)/urdf/_d435.urdf.xacro" />
+    <!-- Аргументы realsense -->
+    <xacro:arg name="use_nominal_extrinsics" default="false"/>
+    <xacro:arg name="add_plug" default="false" />
+    <xacro:arg name="use_mesh" default="true" />
+      <xacro:sensor_d435 parent="big_box_link" use_nominal_extrinsics="$(arg use_nominal_extrinsics)" add_plug="$(arg add_plug)" use_mesh="$(arg use_mesh)">
+      <origin xyz="0.06 0.09 0.018" rpy="0 0.01 0"/>
+      </xacro:sensor_d435>
+  </xacro:if>
 </robot>

Commit message: camera pitch for real

File: src/tracked_description/urdf/t21.urdf.xacro (robot description, xacro)
@@ -39,5 +39,5 @@
     <xacro:arg name="use_mesh" default="true" />
       <xacro:sensor_d435 parent="big_box_link" use_nominal_extrinsics="$(arg use_nominal_extrinsics)" add_plug="$(arg add_plug)" use_mesh="$(arg use_mesh)">
-      <origin xyz="0.06 0.09 0.018" rpy="0 0.01 0"/>
+      <origin xyz="0.06 0.09 0.018" rpy="0 0.015 0"/>
       </xacro:sensor_d435>
   </xacro:if>
