Commit message: second commit

File: src/tracked_description/urdf/tracked_robot.urdf.xacro (robot description, xacro)
@@ -44,12 +44,12 @@
                    scale="${scale_small}"
                    color="${color_grey}"
-                   rpy="-1.57 0 0"
+                   rpy="0 0 0"
                    xyz="0 0 0"/>
   <joint name="geom_joint" type="revolute">
     <parent link="base_link"/>
     <child  link="geom_link"/>
-    <origin xyz="-0.22513 0.1925 0.07335" rpy="0 0 0"/>
-    <axis   xyz="0 1 0"/>
-    <limit lower="-1.57" upper="3.14" effort="1000" velocity="1"/>
+    <origin xyz="-0.22513 -0.1925 0.07335" rpy="1.57 3.14 0"/>
+    <axis   xyz="0 0 1"/>
+    <limit lower="0" upper="3.14" effort="1000" velocity="1"/>
   </joint>
   <!-- ──────────────── VIRTUAL JOINTS FOR SPEEDS ──────────────── -->

Commit message: fourth commit

File: src/tracked_description/urdf/tracked_robot.urdf.xacro (robot description, xacro)
@@ -51,5 +51,5 @@
     <origin xyz="-0.22513 -0.1925 0.07335" rpy="1.57 1.0472 0"/>
     <axis   xyz="0 0 1"/>
-    <limit lower="0" upper="6.25" effort="1000" velocity="1"/>
+    <limit lower="0" upper="3.14" effort="1000" velocity="1"/>
   </joint>
   <!-- ──────────────── VIRTUAL JOINTS FOR SPEEDS ──────────────── -->

Commit message: fifth commit

File: src/tracked_description/urdf/tracked_robot.urdf.xacro (robot description, xacro)
@@ -61,5 +61,5 @@
   <joint name="wheel_left_joint" type="continuous">
     <parent link="base_link"/><child link="wheel_left_link"/>
-    <origin xyz="0 0.19 0.07335" rpy="0 0 0"/>
+    <origin xyz="0 0.17 0.07335" rpy="0 0 0"/>
     <axis   xyz="0 1 0"/>
   </joint>
@@ -71,5 +71,5 @@
   <joint name="wheel_right_joint" type="continuous">
     <parent link="base_link"/><child link="wheel_right_link"/>
-    <origin xyz="0 -0.19 0.07335" rpy="0 0 0"/>
+    <origin xyz="0 -0.17 0.07335" rpy="0 0 0"/>
     <axis   xyz="0 1 0"/>
   </joint>

Commit message: sixth commit

File: src/tracked_description/urdf/tracked_robot.urdf.xacro (robot description, xacro)
@@ -32,5 +32,5 @@
                    scale="${scale_small}"
                    color="${color_grey}"
-                   rpy="1.57 0 0"
+                   rpy="0 0 0"
                    xyz="0 0 0"/>
   <joint name="base_joint" type="fixed">
@@ -49,7 +49,7 @@
     <parent link="base_link"/>
     <child  link="geom_link"/>
-    <origin xyz="-0.22513 -0.1925 0.07335" rpy="1.57 1.0472 0"/>
+    <origin xyz="0.22513 0.1925 0.07335" rpy="-1.57 2.0944 0"/>
     <axis   xyz="0 0 1"/>
-    <limit lower="0" upper="3.14" effort="1000" velocity="1"/>
+    <limit lower="0.174533" upper="5.93412" effort="1000" velocity="1"/>
   </joint>
   <!-- ──────────────── VIRTUAL JOINTS FOR SPEEDS ──────────────── -->

Commit message: seventh commit

File: src/tracked_description/urdf/tracked_robot.urdf.xacro (robot description, xacro)
@@ -3,4 +3,5 @@
   <!-- ──────────────── CONSTANTS ──────────────── -->
   <xacro:property name="scale_small" value="1"/>
+  <xacro:property name="scale_big" value="0.001"/>
   <xacro:property name="color_grey"  value="0.6 0.6 0.6 1.0"/>
   <!-- ──────────────── MACROS ──────────────── -->
@@ -74,3 +75,23 @@
     <axis   xyz="0 1 0"/>
   </joint>
+  <!-- ──────────────── BOX AND SENSORS ──────────────── -->
+  <xacro:add_link  name="big_box_link"
+                   mesh="big_box.stl"
+                   scale="${scale_big}"
+                   color="${color_grey}"
+                   rpy="0 0 0"
+                   xyz="0 0 0"/>
+  <joint name="big_box_joint" type="fixed">
+    <parent link="base_link"/><child link="big_box_link"/>
+    <origin xyz="0.265 -0.093 0.133" rpy="0 0 0"/>
+  </joint>
+  <link name="lidar_link">
+    <inertial><mass value="1e-6"/><origin xyz="0 0 0" rpy="0 0 0"/>
+      <inertia ixx="1e-6" iyy="1e-6" izz="1e-6" ixy="0" ixz="0" iyz="0"/>
+    </inertial>
+  </link>
+  <joint name="lidar_joint" type="fixed">
+    <parent link="big_box_link"/><child link="lidar_link"/>
+    <origin xyz="-0.111 0.092 0.118" rpy="0 0 0"/>
+  </joint>
 </robot>

Commit message: ninth commit

File: src/tracked_description/urdf/tracked_robot.urdf.xacro (robot description, xacro)
@@ -50,5 +50,5 @@
     <parent link="base_link"/>
     <child  link="geom_link"/>
-    <origin xyz="0.22513 0.1925 0.07335" rpy="-1.57 2.0944 0"/>
+    <origin xyz="0.22513 0.1925 0.07335" rpy="-1.57 4.71239 0"/>
     <axis   xyz="0 0 1"/>
     <limit lower="0.174533" upper="5.93412" effort="1000" velocity="1"/>
@@ -62,5 +62,5 @@
   <joint name="wheel_left_joint" type="continuous">
     <parent link="base_link"/><child link="wheel_left_link"/>
-    <origin xyz="0 0.17 0.07335" rpy="0 0 0"/>
+    <origin xyz="0 0.185 0.065" rpy="0 0 0"/>
     <axis   xyz="0 1 0"/>
   </joint>
@@ -72,5 +72,5 @@
   <joint name="wheel_right_joint" type="continuous">
     <parent link="base_link"/><child link="wheel_right_link"/>
-    <origin xyz="0 -0.17 0.07335" rpy="0 0 0"/>
+    <origin xyz="0 -0.185 0.065" rpy="0 0 0"/>
     <axis   xyz="0 1 0"/>
   </joint>

Commit message: try to add sim

File: src/tracked_description/urdf/tracked_robot.urdf.xacro (robot description, xacro)
@@ -62,5 +62,5 @@
   <joint name="wheel_left_joint" type="continuous">
     <parent link="base_link"/><child link="wheel_left_link"/>
-    <origin xyz="0 0.185 0.065" rpy="0 0 0"/>
+    <origin xyz="0 0.1865 0.065" rpy="0 0 0"/>
     <axis   xyz="0 1 0"/>
   </joint>
@@ -72,5 +72,5 @@
   <joint name="wheel_right_joint" type="continuous">
     <parent link="base_link"/><child link="wheel_right_link"/>
-    <origin xyz="0 -0.185 0.065" rpy="0 0 0"/>
+    <origin xyz="0 -0.1865 0.065" rpy="0 0 0"/>
     <axis   xyz="0 1 0"/>
   </joint>

Commit message: fixes to make lio-sam work on 27.11 - TODO make it looks fine and remade structure

File: src/tracked_description/urdf/tracked_robot.urdf.xacro (robot description, xacro)
@@ -5,4 +5,6 @@
   <xacro:property name="scale_big" value="0.001"/>
   <xacro:property name="color_grey"  value="0.6 0.6 0.6 1.0"/>
+  <xacro:t21_ros2_control name="t21" prefix="$(arg prefix)"/>
+  <xacro:include filename="$(find tracked_description)/config/t21.ros2_control.xacro"/>
   <!-- ──────────────── MACROS ──────────────── -->
   <xacro:macro name="add_link" params="name mesh scale color rpy xyz">
@@ -36,6 +38,6 @@
                    xyz="0 0 0"/>
   <joint name="base_joint" type="fixed">
-    <parent link="world"/>
-    <child  link="base_link"/>
+    <parent link="lidar_link"/>
+    <child  link="world"/>
     <origin xyz="0 0 0" rpy="0 0 0"/>
   </joint>
@@ -83,6 +85,6 @@
                    xyz="0 0 0"/>
   <joint name="big_box_joint" type="fixed">
-    <parent link="base_link"/><child link="big_box_link"/>
-    <origin xyz="0.265 -0.093 0.133" rpy="0 0 0"/>
+    <parent link="big_box_link"/><child link="base_link"/>
+    <origin xyz="-0.265 0.093 -0.133" rpy="0 0 0"/>
   </joint>
   <link name="lidar_link">
@@ -92,6 +94,6 @@
   </link>
   <joint name="lidar_joint" type="fixed">
-    <parent link="big_box_link"/><child link="lidar_link"/>
-    <origin xyz="-0.111 0.092 0.118" rpy="0 0 0"/>
+    <parent link="lidar_link"/><child link="big_box_link"/>
+    <origin xyz="0.111 -0.092 -0.118" rpy="0 0 0"/>
   </joint>
 </robot>

Commit message: fine lio-sam and teleop script TODO fix decription

File: src/tracked_description/urdf/tracked_robot.urdf.xacro (robot description, xacro)
@@ -5,6 +5,7 @@
   <xacro:property name="scale_big" value="0.001"/>
   <xacro:property name="color_grey"  value="0.6 0.6 0.6 1.0"/>
+  <xacro:arg name="prefix" default=""/>
+  <xacro:include filename="$(find tracked_description)/config/t21.ros2_control.xacro"/>
   <xacro:t21_ros2_control name="t21" prefix="$(arg prefix)"/>
-  <xacro:include filename="$(find tracked_description)/config/t21.ros2_control.xacro"/>
   <!-- ──────────────── MACROS ──────────────── -->
   <xacro:macro name="add_link" params="name mesh scale color rpy xyz">
@@ -97,3 +98,41 @@
     <origin xyz="0.111 -0.092 -0.118" rpy="0 0 0"/>
   </joint>
+<!--
+  <xacro:macro name="box_inertia" params="b_mass b_length b_width b_height">
+    <inertial>
+      <mass value="${b_mass}"/>
+      <inertia ixx="${(b_mass/12.0) * (b_width*b_width + b_height*b_height)}"
+               ixy="0" ixz="0"
+               iyy="${(b_mass/12.0) * (b_length*b_length + b_height*b_height)}"
+               iyz="0"
+               izz="${(b_mass/12.0) * (b_length*b_length + b_width*b_width)}"/>
+    </inertial>
+  </xacro:macro>
+  <xacro:macro name="xsens_link_geometry">
+    <geometry>
+      <box size="0.001 0.001 0.001"/>
+    </geometry>
+    <origin xyz="0 0 0" rpy="0 0 0"/>
+  </xacro:macro>
+  <link name="imu_link">
+    <visual>
+      <xacro:xsens_link_geometry/>
+      <material name="grey">
+        <color rgba="0.5 0.5 0.5 1"/>
+      </material>
+    </visual>
+    <collision>
+      <xacro:xsens_link_geometry/>
+    </collision>
+    <xacro:box_inertia
+      b_mass="0.1"
+      b_length="0.1"
+      b_width="0.1"
+      b_height="0.1"/>
+  </link>
+  <joint name="xsens_joint" type="fixed">
+    <parent link="laser_link"/>
+    <child link="imu_link"/>
+    <origin xyz="-0.154,  0.0, -0.251" rpy="0 0 0"/>
+  </joint> -->
 </robot>

Commit message: debug

File: src/tracked_description/urdf/tracked_robot.urdf.xacro (robot description, xacro)
@@ -36,6 +36,6 @@
                    xyz="0 0 0"/>
   <joint name="base_joint" type="fixed">
-    <parent link="world"/>
-    <child  link="base_link"/>
+    <parent link="lidar_link"/>
+    <child  link="world"/>
     <origin xyz="0 0 0" rpy="0 0 0"/>
   </joint>
@@ -83,6 +83,6 @@
                    xyz="0 0 0"/>
   <joint name="big_box_joint" type="fixed">
-    <parent link="base_link"/><child link="big_box_link"/>
-    <origin xyz="0.265 -0.093 0.133" rpy="0 0 0"/>
+    <parent link="big_box_link"/><child link="base_link"/>
+    <origin xyz="-0.265 0.093 -0.133" rpy="0 0 0"/>
   </joint>
   <link name="lidar_link">
@@ -92,6 +92,6 @@
   </link>
   <joint name="lidar_joint" type="fixed">
-    <parent link="big_box_link"/><child link="lidar_link"/>
-    <origin xyz="-0.111 0.092 0.118" rpy="0 0 0"/>
+    <parent link="lidar_link"/><child link="big_box_link"/>
+    <origin xyz="0.111 -0.092 -0.118" rpy="0 0 0"/>
   </joint>
 </robot>
