Commit message: changed params, camera setup t simulate cuVSLAM

File: src/tracked_description/urdf/camera.xacro (robot description, xacro)
@@ -1,6 +1,6 @@
 <?xml version="1.0"?>
 <robot xmlns:xacro="http://www.ros.org/wiki/xacro" >
-    <xacro:property name="camera_translation" value="0.06 0.09 0.018"/>
-    <xacro:arg name="depth" default="true"/>
+  <xacro:property name="camera_translation" value="0.06 0.09 0.018"/>
+  <xacro:unless value = "$(arg use_sim_time)">
     <xacro:include filename="$(find realsense2_description)/urdf/_d435.urdf.xacro"/>
     <!-- Аргументы realsense -->
@@ -12,16 +12,63 @@
       <origin xyz="${camera_translation}" rpy="0 0.015 0"/>
     </xacro:sensor_d435>
-    <xacro:if value="$(arg use_sim_time)">
-        <xacro:if value="$(arg depth)">
-            <gazebo reference="camera_link">
-                <material>Gazebo/Red</material>
-                <sensor name="camera" type="depth">
-                <pose> 0 0 0 0 0 0 </pose>
-                <visualize>true</visualize>
+  </xacro:unless>
+  <xacro:if value="$(arg use_sim_time)">
+    <xacro:arg name="depth" default="false"/>
+      <xacro:macro name="add_camera" params="name xyz">
+          <link name="${name}_link"/>
+          <joint name="${name}_joint" type="fixed">
+            <parent link="big_box_link"/>
+            <child link="${name}_link"/>
+            <origin xyz="${xyz}" rpy="0.0 0.0 0.0"/>
+          </joint>
+          <link name="${name}_optical_link"/>
+          <joint name="${name}_optical_joint" type="fixed">
+            <parent link="${name}_link"/>
+            <child link="${name}_optical_link"/>
+            <origin xyz="0.0 0.0 0.0" rpy="${-pi/2} 0 ${-pi/2}"/>
+          </joint>
+      </xacro:macro>
+      <xacro:if value="$(arg depth)">
+          <gazebo reference="camera_link">
+              <material>Gazebo/Red</material>
+              <sensor name="camera" type="depth">
+              <pose> 0 0 0 0 0 0 </pose>
+              <visualize>true</visualize>
+              <update_rate>10</update_rate>
+              <camera>
+                  <horizontal_fov>1.089</horizontal_fov>
+                  <image>
+                      <format>B8G8R8</format>
+                      <width>640</width>
+                      <height>480</height>
+                  </image>
+                  <clip>
+                      <near>0.05</near>
+                      <far>8.0</far>
+                  </clip>
+              </camera>
+              <plugin name="camera_controller" filename="libgazebo_ros_camera.so">
+                  <!-- TODO Fix argument dependency -->
+                  <frame_name>camera_depth_optical_frame</frame_name>
+                  <min_depth>0.1</min_depth>
+                  <max_depth>100.0</max_depth>
+                  </plugin>
+              </sensor>
+          </gazebo>
+      </xacro:if>
+      <xacro:unless value="$(arg depth)">
+        <xacro:add_camera name='camera_1' xyz="${camera_translation}"/>
+        <xacro:add_camera name='camera_2' xyz="0.06 0.12 0.018"/>
+        <!-- Камера infra1 -->
+        <gazebo reference="camera_1_link">
+            <material>Gazebo/Red</material>
+            <sensor name="camera/infra1" type="camera">
+                <pose> 0.0 0.0 0.0 0 0 0 </pose>
+                <visualize>false</visualize>
                 <update_rate>10</update_rate>
                 <camera>
                     <horizontal_fov>1.089</horizontal_fov>
                     <image>
-                        <format>B8G8R8</format>
+                        <format>R8G8B8</format>
                         <width>640</width>
                         <height>480</height>
@@ -29,41 +76,85 @@
                     <clip>
                         <near>0.05</near>
-                        <far>8.0</far>
+                        <far>15.0</far>
                     </clip>
                 </camera>
-                <plugin name="camera_controller" filename="libgazebo_ros_camera.so">
-                    <!-- TODO Fix argument dependency -->
-                    <frame_name>camera_depth_optical_frame</frame_name>
-                    <min_depth>0.1</min_depth>
-                    <max_depth>100.0</max_depth>
-                    </plugin>
-                </sensor>
-            </gazebo>
-        </xacro:if>
-        <xacro:unless value="$(arg depth)">
-            <gazebo reference="front_camera_link">
-                <material>Gazebo/Red</material>
-                <sensor name="camera" type="camera">
-                    <pose> 0 0 0 0 0 0 </pose>
-                    <visualize>true</visualize>
-                    <update_rate>10</update_rate>
-                    <camera>
-                        <horizontal_fov>1.089</horizontal_fov>
-                        <image>
-                            <format>R8G8B8</format>
-                            <width>640</width>
-                            <height>480</height>
-                        </image>
-                        <clip>
-                            <near>0.05</near>
-                            <far>8.0</far>
-                        </clip>
-                    </camera>
-                    <plugin name="camera_controller" filename="libgazebo_ros_camera.so">
-                        <frame_name>camera_depth_optical_frame</frame_name>
-                    </plugin>
-                </sensor>
-            </gazebo>
-        </xacro:unless>
-    </xacro:if>
+                <plugin name="camera_controller_infra1" filename="libgazebo_ros_camera.so">
+                    <frameName>camera_1_optical_link</frameName>
+                    <cameraName>camera/infra1</cameraName>
+                    <imageTopicName>image_rect_raw</imageTopicName>
+                    <cameraInfoTopicName>camera_info</cameraInfoTopicName>
+                    <minDepth>0.1</minDepth>
+                    <maxDepth>100.0</maxDepth>
+                </plugin>
+            </sensor>
+        </gazebo>
+        <!-- Камера infra2 -->
+        <gazebo reference="camera_2_link">
+            <material>Gazebo/Orange</material>
+            <sensor name="camera/infra2" type="camera">
+                <pose> 0.0 0.0 0.0 0 0 0 </pose>  <!-- Смещение 3 см по Y для второй камеры -->
+                <visualize>false</visualize>
+                <update_rate>10</update_rate>
+                <camera>
+                    <horizontal_fov>1.089</horizontal_fov>
+                    <image>
+                        <format>R8G8B8</format>
+                        <width>640</width>
+                        <height>480</height>
+                    </image>
+                    <clip>
+                        <near>0.05</near>
+                        <far>15.0</far>
+                    </clip>
+                </camera>
+                <plugin name="camera_controller_infra2" filename="libgazebo_ros_camera.so">
+                    <frameName>camera_2_optical_link</frameName>
+                    <cameraName>camera/infra2</cameraName>
+                    <imageTopicName>image_rect_raw</imageTopicName>
+                    <cameraInfoTopicName>camera_info</cameraInfoTopicName>
+                    <minDepth>0.1</minDepth>
+                    <maxDepth>100.0</maxDepth>
+                </plugin>
+            </sensor>
+        </gazebo>
+        <link name="imu_camera_link">
+          <visual>
+            <geometry>
+              <box size="0.001 0.001 0.001"/>
+            </geometry>
+            <material name="blue">
+              <color rgba="0.0 0.0 1.0 0.5"/>
+            </material>
+          </visual>
+          <inertial>
+            <mass value="0.01"/>
+            <inertia ixx="0.00001" ixy="0.0" ixz="0.0"
+                     iyy="0.00001" iyz="0.0"
+                     izz="0.00001"/>
+          </inertial>
+        </link>
+        <joint name="imu_camera_joint" type="fixed">
+          <parent link="camera_1_link"/>
+          <child link="imu_camera_link"/>
+          <origin xyz="0.0 0.00 0.00" rpy="0 0 0"/>
+        </joint>
+        <gazebo reference="imu_camera_link">
+          <gravity>true</gravity>
+          <sensor name="imu_camera_sensor" type="imu">
+            <pose relative_to='imu_camera_link'>0 0 0 0 0 0</pose>
+            <always_on>true</always_on>
+            <update_rate>100</update_rate>
+            <plugin filename="libgazebo_ros_imu_sensor.so" name="camera_imu_plugin">
+              <ros>
+                <remapping>~/out:=/camera/imu/data</remapping>
+              </ros>
+              <frameName>imu_camera_link</frameName>
+              <topicName>camera/imu/data</topicName>
+              <bodyName>imu_camera_link</bodyName>
+              <initialOrientationAsReference>false</initialOrientationAsReference>
+            </plugin>
+          </sensor>
+        </gazebo>
+      </xacro:unless>
+  </xacro:if>
 </robot>

File: src/tracked_description/urdf/imu.xacro (robot description, xacro)
@@ -59,6 +59,8 @@
           <gaussianNoise>0.001</gaussianNoise>
           <xyzOffset>0 0 0</xyzOffset>
-          <rpyOffset>0 0 0</rpyOffset>
-          <frameName>xsens_link</frameName-->
+          <rpyOffset>0 0 0</rpyOffset>-->
+          <frameName>imu_link</frameName>
+          <bodyName>imu_link</bodyName>
+          <initialOrientationAsReference>false</initialOrientationAsReference>
         </plugin>
       </sensor>

File: src/tracked_description/urdf/lidar.xacro (robot description, xacro)
@@ -29,6 +29,6 @@
       max_range="25.0"
       noise="0.0"
-      min_angle="-${pi/2}"
-      max_angle="${pi/2}"
+      min_angle="-${pi}"
+      max_angle="${pi}"
       gpu="false">
       <origin xyz="0 0 -0.035" rpy="0 0 0" />
