Commit message: change imu topic and camera roll

File: src/t21_sim/urdf/imu.xacro (robot description, xacro)
@@ -51,5 +51,5 @@
       <plugin filename="libgazebo_ros_imu_sensor.so" name="imu_plugin">
         <ros>
-          <remapping>~/out:=/imu/data</remapping>
+          <remapping>~/out:=/imu/data_raw</remapping>
         </ros>
         <!--topicName>imu/data_raw</topicName>

File: src/t21_sim/urdf/t21.urdf.xacro (robot description, xacro)
@@ -28,5 +28,5 @@
   <xacro:arg name="use_mesh" default="true" />
   <xacro:sensor_d435 parent="big_box_link" use_nominal_extrinsics="$(arg use_nominal_extrinsics)" add_plug="$(arg add_plug)" use_mesh="$(arg use_mesh)">
-    <origin xyz="0.06 0.09 0.018" rpy="0 0.01 0"/>
+    <origin xyz="0.06 0.09 0.018" rpy="0 0.015 0"/>
   </xacro:sensor_d435>
   <xacro:include filename="$(find t21_sim)/urdf/depth_camera.xacro" />

Commit message: try to add lio-sam

File: src/t21_sim/urdf/imu.xacro (robot description, xacro)
@@ -48,5 +48,5 @@
       <pose relative_to='xsens_link'>0 0 0 0 0 0</pose>
       <always_on>true</always_on>
-      <update_rate>100</update_rate>
+      <update_rate>10</update_rate>
       <plugin filename="libgazebo_ros_imu_sensor.so" name="imu_plugin">
         <ros>

File: src/tracked_description/urdf/tracked_robot.urdf.xacro (robot description, xacro)
@@ -86,4 +86,17 @@
     <origin xyz="0.265 -0.093 0.133" rpy="0 0 0"/>
   </joint>
+  <!-- ──────────────── IMU LINK ──────────────── -->
+  <link name="imu_link">
+    <inertial>
+      <mass value="0.01"/>
+      <origin xyz="0 0 0" rpy="0 0 0"/>
+      <inertia ixx="1e-6" iyy="1e-6" izz="1e-6" ixy="0" ixz="0" iyz="0"/>
+    </inertial>
+  </link>
+  <joint name="imu_joint" type="fixed">
+    <parent link="big_box_link"/>
+    <child link="imu_link"/>
+    <origin xyz="0 0 0" rpy="0 0 0"/>
+  </joint>
   <link name="lidar_link">
     <inertial><mass value="1e-6"/><origin xyz="0 0 0" rpy="0 0 0"/>
