Commit message: Added camera & lidar description, modified launch to bringup entire stack

File: src/t21_sim/urdf/t21.urdf.xacro (robot description, xacro)
@@ -6,3 +6,29 @@
   <!-- блок ros2_control -->
   <xacro:include filename="$(find t21_sim)/config/t21.ros2_control.xacro"/>
+    <!-- блок симуляции VLP-16-->
+  <xacro:include filename="$(find velodyne_description)/urdf/VLP-16.urdf.xacro"/>
+  <xacro:VLP-16 parent="lidar_link"
+                name="velodyne"
+                topic="/velodyne_points"
+                organize_cloud="true"
+                hz="10"
+                lasers="8"
+                samples="400"
+                min_range="0.5"
+                max_range="25.0"
+                min_angle="-3.14159265359"
+                max_angle="3.14159265359"
+                gpu="false">
+                <origin xyz="0 0 -0.04" rpy="0 0 0" />
+   </xacro:VLP-16>
+  <xacro:include filename="$(find realsense2_description)/urdf/_d435.urdf.xacro" />
+  <!-- Аргументы realsense -->
+  <!-- TODO change camera pith to match real one -->
+  <xacro:arg name="use_nominal_extrinsics" default="false"/>
+  <xacro:arg name="add_plug" default="false" />
+  <xacro:arg name="use_mesh" default="true" />
+  <xacro:sensor_d435 parent="big_box_link" use_nominal_extrinsics="$(arg use_nominal_extrinsics)" add_plug="$(arg add_plug)" use_mesh="$(arg use_mesh)">
+    <origin xyz="0.06 0.09 0.018" rpy="0 0.01 0"/>
+  </xacro:sensor_d435>
+  <xacro:include filename="$(find t21_sim)/urdf/depth_camera.xacro" />
 </robot>

Commit message: fix urdf for new control box

File: src/t21_sim/urdf/t21.urdf.xacro (robot description, xacro)
@@ -19,5 +19,5 @@
                 max_angle="3.14159265359"
                 gpu="false">
-                <origin xyz="0 0 -0.04" rpy="0 0 0" />
+                <origin xyz="0 0 0" rpy="0 0 0" />
    </xacro:VLP-16>
   <xacro:include filename="$(find realsense2_description)/urdf/_d435.urdf.xacro" />

File: src/t21_sim/urdf/tracked_robot.urdf.xacro (robot description, xacro)
@@ -122,6 +122,5 @@
         <origin rpy="0 0 0" xyz="0 0 0"/>
         <geometry>
-          <mesh filename="file://$(find t21_sim)/meshes/big_box.stl"
-                scale="0.001 0.001 0.001"/>
+          <mesh filename="file://$(find t21_sim)/meshes/control_box.STL"/>
         </geometry>
       </collision>
@@ -129,6 +128,5 @@
         <origin rpy="0 0 0" xyz="0 0 0"/>
         <geometry>
-          <mesh filename="file://$(find t21_sim)/meshes/big_box.stl"
-                scale="0.001 0.001 0.001"/>
+          <mesh filename="file://$(find t21_sim)/meshes/control_box.STL"/>
         </geometry>
         <material name="light_blue"/>
@@ -137,5 +135,5 @@
   <joint name="big_box_joint" type="fixed">
     <parent link="base_link"/><child link="big_box_link"/>
-    <origin xyz="0.265 -0.093 0.1" rpy="0 0 0"/>
+    <origin xyz="0.165 0.0 0.104" rpy="0 0 0"/>
   </joint>
   <!-- Gazebo extensions -->

File: src/tracked_description/urdf/lidar.xacro (robot description, xacro)
@@ -1,5 +1,5 @@
 <?xml version="1.0"?>
 <robot xmlns:xacro="http://www.ros.org/wiki/xacro">
-  <xacro:property name="lidar_translation" value="-0.111 0.092 0.118"/>
+  <xacro:property name="lidar_translation" value="0.0036 -2.29E-05 0.095"/>
     <link name="lidar_link">
       <inertial>
@@ -32,5 +32,5 @@
       max_angle="${pi}"
       gpu="false">
-      <origin xyz="0 0 -0.035" rpy="0 0 0" />
+      <origin xyz="0 0 0" rpy="0 0 0" />
     </xacro:VLP-16>
   </xacro:if>

File: src/tracked_description/urdf/tracked_robot.urdf.xacro (robot description, xacro)
@@ -77,6 +77,6 @@
   <!-- ──────────────── BOX AND SENSORS ──────────────── -->
   <xacro:add_link  name="big_box_link"
-                   mesh="big_box.stl"
-                   scale="${scale_big}"
+                   mesh="control_box.STL"
+                   scale="${scale_small}"
                    color="${color_grey}"
                    rpy="0 0 0"
@@ -85,5 +85,5 @@
     <parent link="base_link"/>
     <child link="big_box_link"/>
-    <origin xyz="0.265 -0.093 0.133" rpy="0 0 0"/>
+    <origin xyz="0.165 0.0 0.139" rpy="0 0 0"/>
   </joint>
 </robot>
