Commit message: add fliper working joint

File: src/t21_sim/urdf/tracked_robot.urdf.xacro (robot description, xacro)
@@ -116,5 +116,5 @@
     <child link="fliper_link"/>
     <axis xyz="0 -1 0"/>
-    <limit lower="0" upper="0" effort="10" velocity="10"/>
+    <limit lower="0.174533" upper="5.93412" effort="1000" velocity="1"/>
   </joint>
   <link name="big_box_link">

Commit message: add motion_emulator

File: src/t21_sim/urdf/tracked_robot.urdf.xacro (robot description, xacro)
@@ -112,5 +112,5 @@
   </link>
   <joint name="fliper_joint" type="revolute">
-    <origin xyz="0.222 0.2435 0.04" rpy="0 0 0"/>
+    <origin xyz="0.222 0.2435 0.04" rpy="0 3.25 0"/>
     <parent link="base_link"/>
     <child link="fliper_link"/>

Commit message: succesfull merge tms and oka branch, working sim mode

File: src/t21_sim/urdf/tracked_robot.urdf.xacro (robot description, xacro)
@@ -11,4 +11,5 @@
     <color rgba="0.79216 0.81961 0.93333 1"/>
   </material>
+  <link name="root_link"/>
   <!-- Base Link -->
   <link name="base_link">
@@ -32,4 +33,9 @@
     </collision>
   </link>
+  <joint name="root_joint" type="fixed">
+    <parent link="root_link"/>
+    <child link="base_link"/>
+    <origin xyz="0 0 0" rpy="0 0 0"/>
+  </joint>
   <!-- Left Wheel -->
   <link name="left_wheel_link">

Commit message: united description and launch for real robot and sim

File: src/t21_sim/urdf/tracked_robot.urdf.xacro (robot description, xacro)
@@ -33,5 +33,5 @@
   </link>
   <!-- Left Wheel -->
-  <link name="left_wheel_link">
+  <link name="wheel_left_link">
     <inertial>
       <origin xyz="0 -0.015 0" rpy="0 0 0"/>
@@ -53,8 +53,8 @@
     </collision>
   </link>
-  <joint name="left_wheel_joint" type="continuous">
+  <joint name="wheel_left_joint" type="continuous">
     <origin xyz="-0.015028 0.2025 0.04" rpy="0 0 0"/>
     <parent link="base_link"/>
-    <child link="left_wheel_link"/>
+    <child link="wheel_left_link"/>
     <axis xyz="0 1 0"/>
     <limit effort="10" velocity="10"/>
@@ -62,5 +62,5 @@
   </joint>
   <!-- Right Wheel -->
-  <link name="right_wheel_link">
+  <link name="wheel_right_link">
     <inertial>
       <origin xyz="0 0.015 0" rpy="0 0 0"/>
@@ -82,8 +82,8 @@
     </collision>
   </link>
-  <joint name="right_wheel_joint" type="continuous">
+  <joint name="wheel_right_joint" type="continuous">
     <origin xyz="-0.015028 -0.2025 0.04" rpy="0 0 0"/>
     <parent link="base_link"/>
-    <child link="right_wheel_link"/>
+    <child link="wheel_right_link"/>
     <axis xyz="0 1 0"/>
     <limit effort="10" velocity="10"/>
@@ -139,13 +139,4 @@
     <origin xyz="0.265 -0.093 0.1" rpy="0 0 0"/>
   </joint>
-  <link name="lidar_link">
-    <inertial><mass value="1e-6"/><origin xyz="0 0 0" rpy="0 0 0"/>
-      <inertia ixx="1e-6" iyy="1e-6" izz="1e-6" ixy="0" ixz="0" iyz="0"/>
-    </inertial>
-  </link>
-  <joint name="lidar_joint" type="fixed">
-    <parent link="big_box_link"/><child link="lidar_link"/>
-    <origin xyz="-0.111 0.092 0.118" rpy="0 0 0"/>
-  </joint>
   <!-- Gazebo extensions -->
   <gazebo reference="base_link">

File: src/tracked_description/config/t21.ros2_control.xacro (robot description, xacro)
@@ -6,13 +6,48 @@
        несколько роботов в одном графе.
   ================================================================= -->
-  <xacro:macro name="t21_ros2_control" params="name prefix">
-    <ros2_control name="${name}_hw" type="system">
+  <xacro:unless value="$(arg use_sim_time)">
+    <xacro:macro name="t21_ros2_control" params="name prefix">
+      <ros2_control name="${name}_hw" type="system">
+        <!-- аппаратный плагин -->
+        <hardware>
+          <plugin>t21_hardware/T21TrackedHardware</plugin>
+          <!-- при необходимости можно добавить <param …/> -->
+        </hardware>
+        <!-- виртуальный сустав линейной скорости -->
+        <joint name="${prefix}wheel_left_joint">
+          <command_interface name="velocity"/>
+          <state_interface   name="velocity"/>
+          <state_interface name="position"/>
+        </joint>
+        <!-- виртуальный сустав угловой скорости -->
+        <joint name="${prefix}wheel_right_joint">
+          <command_interface name="velocity"/>
+          <state_interface   name="velocity"/>
+          <state_interface name="position"/>
+        </joint>
+        <!-- реальный сустав флиппера / стрелы -->
+        <joint name="${prefix}flipper_joint">
+          <command_interface name="position"/>
+          <state_interface   name="position"/>
+        </joint>
+      </ros2_control>
+    </xacro:macro>
+    <!-- Вызываем макрос, передавая имя и префикс -->
+    <xacro:t21_ros2_control name="t21" prefix="$(arg prefix)"/>
+  </xacro:unless>
+  <xacro:if value="$(arg use_sim_time)">
+    <!-- ===========================================================
+       Определяем ROS 2 Control-блок для гусеничной платформы Т-21
+       Параметр prefix (по-умолчанию пустой) позволяет запускать
+       несколько роботов в одном графе.
+    ================================================================= -->
+    <ros2_control name="GazeboSystem" type="system">
       <!-- аппаратный плагин -->
       <hardware>
-        <plugin>t21_hardware/T21TrackedHardware</plugin>
+        <plugin>gazebo_ros2_control/GazeboSystem</plugin>
         <!-- при необходимости можно добавить <param …/> -->
       </hardware>
       <!-- виртуальный сустав линейной скорости -->
-      <joint name="${prefix}wheel_left_joint">
+      <joint name="wheel_left_joint">
         <command_interface name="velocity"/>
         <state_interface   name="velocity"/>
@@ -20,15 +55,24 @@
       </joint>
       <!-- виртуальный сустав угловой скорости -->
-      <joint name="${prefix}wheel_right_joint">
+      <joint name="wheel_right_joint">
         <command_interface name="velocity"/>
         <state_interface   name="velocity"/>
         <state_interface name="position"/>
       </joint>
-      <!-- реальный сустав флиппера / стрелы -->
-      <joint name="${prefix}geom_joint">
+      <!--реальный сустав флиппера / стрелы -->
+      <joint name="fliper_joint">
         <command_interface name="position"/>
         <state_interface   name="position"/>
       </joint>
     </ros2_control>
-  </xacro:macro>
+    <gazebo>
+        <plugin name="gazebo_ros2_control" filename="libgazebo_ros2_control.so">
+            <parameters>$(find t21_sim)/config/my_controllers.yaml</parameters>
+        </plugin>
+        <!-- <updateRate>10</updateRate> -->
+        <!-- <ros>
+          <remapping>odom:=odom/unfiltered</remapping>
+        </ros> -->
+    </gazebo>
+  </xacro:if>
 </robot>

File: src/tracked_description/urdf/t21.urdf.xacro (robot description, xacro)
@@ -3,42 +3,20 @@
   <!-- Объявляем аргументы -->
   <xacro:arg name="prefix" default=""/>
-  <!-- Использовать симуляцию лидара\камеры -->
-  <xacro:arg name="sim_lidar" default="false"/>
-  <xacro:arg name="sim_cam" default="true"/>
-  <!-- геометрия -->
-  <xacro:include filename="$(find tracked_description)/urdf/tracked_robot.urdf.xacro"/>
-  <!-- блок ros2_control -->
+  <!-- Использовать симуляцию -->
+  <xacro:arg name="use_sim_time" default="false"/>
+  <!-- Геометрия -->
+  <xacro:unless value="$(arg use_sim_time)">
+    <xacro:include filename="$(find tracked_description)/urdf/tracked_robot.urdf.xacro"/>
+  </xacro:unless>
+  <xacro:if value="$(arg use_sim_time)">
+    <xacro:include filename="$(find t21_sim)/urdf/tracked_robot.urdf.xacro"/>
+  </xacro:if>
+  <!-- Блок ros2_control -->
   <xacro:include filename="$(find tracked_description)/config/t21.ros2_control.xacro"/>
-  <!-- вызываем макрос, передавая имя и префикс -->
-  <xacro:t21_ros2_control name="t21" prefix="$(arg prefix)"/>
-  <!-- Используем свойство вместо прямого аргумента -->
-  <xacro:if value="${'$(arg sim_lidar)' == 'true'}">
-    <!-- блок симуляции VLP-16-->
-    <xacro:include filename="$(find velodyne_description)/urdf/VLP-16.urdf.xacro"/>
-    <xacro:VLP-16 parent="lidar_link"
-                name="velodyne"
-                topic="/velodyne_points"
-                organize_cloud="false"
-                hz="10"
-                lasers="16"
-                samples="400"
-                min_range="0.1"
-                max_range="25.0"
-                min_angle="-1.5708"
-                max_angle="1.5708"
-                gpu="false">
-      <origin xyz="0 0 0" rpy="0 0 0" />
-    </xacro:VLP-16>
-  </xacro:if>
-  <xacro:if value="${'$(arg sim_cam)' == 'true'}">
-    <xacro:include filename="$(find realsense2_description)/urdf/_d435.urdf.xacro" />
-    <!-- Аргументы realsense -->
-    <!-- TODO change camera pith to match real one -->
-    <xacro:arg name="use_nominal_extrinsics" default="false"/>
-    <xacro:arg name="add_plug" default="false" />
-    <xacro:arg name="use_mesh" default="true" />
-      <xacro:sensor_d435 parent="big_box_link" use_nominal_extrinsics="$(arg use_nominal_extrinsics)" add_plug="$(arg add_plug)" use_mesh="$(arg use_mesh)">
-      <origin xyz="0.06 0.09 0.018" rpy="0 0.015 0"/>
-      </xacro:sensor_d435>
-  </xacro:if>
+  <!-- Блок описания LiDAR -->
+  <xacro:include filename="$(find tracked_description)/urdf/lidar.xacro"/>
+  <!-- Блок описания камеры -->
+  <xacro:include filename="$(find tracked_description)/urdf/camera.xacro"/>
+  <!-- Блок описания IMU -->
+  <xacro:include filename="$(find tracked_description)/urdf/imu.xacro"/>
 </robot>

File: src/tracked_description/urdf/tracked_robot.urdf.xacro (robot description, xacro)
@@ -5,7 +5,4 @@
   <xacro:property name="scale_big" value="0.001"/>
   <xacro:property name="color_grey"  value="0.6 0.6 0.6 1.0"/>
-  <xacro:arg name="prefix" default=""/>
-  <xacro:include filename="$(find tracked_description)/config/t21.ros2_control.xacro"/>
-  <xacro:t21_ros2_control name="t21" prefix="$(arg prefix)"/>
   <!-- ──────────────── MACROS ──────────────── -->
   <xacro:macro name="add_link" params="name mesh scale color rpy xyz">
@@ -14,5 +11,5 @@
         <origin rpy="${rpy}" xyz="${xyz}"/>
         <geometry>
-          <mesh filename="package://tracked_description/mesh/${mesh}"
+          <mesh filename="file://$(find tracked_description)/mesh/${mesh}"
                 scale="${scale} ${scale} ${scale}"/>
         </geometry>
@@ -21,5 +18,5 @@
         <origin rpy="${rpy}" xyz="${xyz}"/>
         <geometry>
-          <mesh filename="package://tracked_description/mesh/${mesh}"
+          <mesh filename="file://$(find tracked_description)/mesh/${mesh}"
                 scale="${scale} ${scale} ${scale}"/>
         </geometry>
@@ -30,5 +27,4 @@
     </link>
   </xacro:macro>
-  <link name="world"/>
   <!-- ──────────────── BASE ──────────────── -->
   <xacro:add_link  name="base_link"
@@ -38,11 +34,6 @@
                    rpy="0 0 0"
                    xyz="0 0 0"/>
-  <joint name="base_joint" type="fixed">
-    <parent link="lidar_link"/>
-    <child  link="world"/>
-    <origin xyz="0 0 0" rpy="0 0 0"/>
-  </joint>
   <!-- ──────────────── FLIPPER / GEOMETRY ──────────────── -->
-  <xacro:add_link  name="geom_link"
+  <xacro:add_link  name="flipperlink"
                    mesh="fliper.stl"
                    scale="${scale_small}"
@@ -50,7 +41,7 @@
                    rpy="0 0 0"
                    xyz="0 0 0"/>
-  <joint name="geom_joint" type="revolute">
+  <joint name="flipper_joint" type="revolute">
     <parent link="base_link"/>
-    <child  link="geom_link"/>
+    <child  link="flipper_link"/>
     <origin xyz="0.22513 0.1925 0.07335" rpy="-1.57 4.71239 0"/>
     <axis   xyz="0 0 1"/>
@@ -59,20 +50,26 @@
   <!-- ──────────────── VIRTUAL JOINTS FOR SPEEDS ──────────────── -->
   <link name="wheel_left_link">
-    <inertial><mass value="1e-6"/><origin xyz="0 0 0" rpy="0 0 0"/>
+    <inertial>
+      <mass value="1e-6"/>
+      <origin xyz="0 0 0" rpy="0 0 0"/>
       <inertia ixx="1e-6" iyy="1e-6" izz="1e-6" ixy="0" ixz="0" iyz="0"/>
     </inertial>
   </link>
   <joint name="wheel_left_joint" type="continuous">
-    <parent link="base_link"/><child link="wheel_left_link"/>
+    <parent link="base_link"/>
+    <child link="wheel_left_link"/>
     <origin xyz="0 0.1865 0.065" rpy="0 0 0"/>
     <axis   xyz="0 1 0"/>
   </joint>
   <link name="wheel_right_link">
-    <inertial><mass value="1e-6"/><origin xyz="0 0 0" rpy="0 0 0"/>
+    <inertial>
+    <mass value="1e-6"/>
+    <origin xyz="0 0 0" rpy="0 0 0"/>
       <inertia ixx="1e-6" iyy="1e-6" izz="1e-6" ixy="0" ixz="0" iyz="0"/>
     </inertial>
   </link>
   <joint name="wheel_right_joint" type="continuous">
-    <parent link="base_link"/><child link="wheel_right_link"/>
+    <parent link="base_link"/>
+    <child link="wheel_right_link"/>
     <origin xyz="0 -0.1865 0.065" rpy="0 0 0"/>
     <axis   xyz="0 1 0"/>
@@ -86,53 +83,7 @@
                    xyz="0 0 0"/>
   <joint name="big_box_joint" type="fixed">
-    <parent link="big_box_link"/><child link="base_link"/>
-    <origin xyz="-0.265 0.093 -0.133" rpy="0 0 0"/>
+    <parent link="base_link"/>
+    <child link="big_box_link"/>
+    <origin xyz="0.265 -0.093 0.133" rpy="0 0 0"/>
   </joint>
-  <link name="lidar_link">
-    <inertial><mass value="1e-6"/><origin xyz="0 0 0" rpy="0 0 0"/>
-      <inertia ixx="1e-6" iyy="1e-6" izz="1e-6" ixy="0" ixz="0" iyz="0"/>
-    </inertial>
-  </link>
-  <joint name="lidar_joint" type="fixed">
-    <parent link="lidar_link"/><child link="big_box_link"/>
-    <origin xyz="0.111 -0.092 -0.118" rpy="0 0 0"/>
-  </joint>
-<!--
-  <xacro:macro name="box_inertia" params="b_mass b_length b_width b_height">
-    <inertial>
-      <mass value="${b_mass}"/>
-      <inertia ixx="${(b_mass/12.0) * (b_width*b_width + b_height*b_height)}"
-               ixy="0" ixz="0"
-               iyy="${(b_mass/12.0) * (b_length*b_length + b_height*b_height)}"
-               iyz="0"
-               izz="${(b_mass/12.0) * (b_length*b_length + b_width*b_width)}"/>
-    </inertial>
-  </xacro:macro>
-  <xacro:macro name="xsens_link_geometry">
-    <geometry>
-      <box size="0.001 0.001 0.001"/>
-    </geometry>
-    <origin xyz="0 0 0" rpy="0 0 0"/>
-  </xacro:macro>
-  <link name="imu_link">
-    <visual>
-      <xacro:xsens_link_geometry/>
-      <material name="grey">
-        <color rgba="0.5 0.5 0.5 1"/>
-      </material>
-    </visual>
-    <collision>
-      <xacro:xsens_link_geometry/>
-    </collision>
-    <xacro:box_inertia
-      b_mass="0.1"
-      b_length="0.1"
-      b_width="0.1"
-      b_height="0.1"/>
-  </link>
-  <joint name="xsens_joint" type="fixed">
-    <parent link="laser_link"/>
-    <child link="imu_link"/>
-    <origin xyz="-0.154,  0.0, -0.251" rpy="0 0 0"/>
-  </joint> -->
 </robot>

Commit message: delete lio-sam package with scan context. Can't set up and run and haven't ehough arguments to improve localization

File: src/t21_sim/urdf/tracked_robot.urdf.xacro (robot description, xacro)
@@ -137,4 +137,57 @@
     <origin xyz="0.165 0.0 0.104" rpy="0 0 0"/>
   </joint>
+  <link
+    name="camera_base_link">
+    <inertial>
+      <origin
+        xyz="0.00236723430443658 0.00284830369666845 1.86648075149107E-05"
+        rpy="0 0 0" />
+      <mass
+        value="0.0798291622805554" />
+      <inertia
+        ixx="0.000122650398243472"
+        ixy="-5.35688945763538E-07"
+        ixz="4.40692500921343E-08"
+        iyy="2.06507530748284E-05"
+        iyz="-5.04471506920737E-08"
+        izz="0.000119910604769246" />
+    </inertial>
+    <visual>
+      <origin
+        xyz="0 0 0"
+        rpy="0 0 0" />
+      <geometry>
+        <mesh
+          filename="file://$(find t21_sim)/meshes/camera_base_link.STL" />
+      </geometry>
+      <material
+        name="">
+        <color
+          rgba="0.749019607843137 0.749019607843137 0.749019607843137 1" />
+      </material>
+    </visual>
+    <collision>
+      <origin
+        xyz="0 0 0"
+        rpy="0 0 0" />
+      <geometry>
+        <mesh
+          filename="file://$(find t21_sim)/meshes/camera_base_link.STL" />
+      </geometry>
+    </collision>
+  </link>
+  <joint
+    name="camera_joint"
+    type="fixed">
+    <origin
+      xyz="0.148648549421411 -0.00168373549133136 0.0396301545012917"
+      rpy="0 0 0" />
+    <parent
+      link="big_box_link" />
+    <child
+      link="camera_base_link" />
+    <axis
+      xyz="0 0 0" />
+  </joint>
   <!-- Gazebo extensions -->
   <gazebo reference="base_link">
