Commit message: third commit

File: src/tracked_description/config/t21.ros2_control.xacro (robot description, xacro)
@@ -14,5 +14,5 @@
       </hardware>
       <!-- виртуальный сустав линейной скорости -->
-      <joint name="${prefix}lin_vel_joint">
+      <joint name="${prefix}wheel_left_joint">
         <command_interface name="velocity"/>
         <state_interface   name="velocity"/>
@@ -20,5 +20,5 @@
       </joint>
       <!-- виртуальный сустав угловой скорости -->
-      <joint name="${prefix}ang_vel_joint">
+      <joint name="${prefix}wheel_right_joint">
         <command_interface name="velocity"/>
         <state_interface   name="velocity"/>

File: src/tracked_description/urdf/tracked_robot.urdf.xacro (robot description, xacro)
@@ -49,28 +49,28 @@
     <parent link="base_link"/>
     <child  link="geom_link"/>
-    <origin xyz="-0.22513 -0.1925 0.07335" rpy="1.57 3.14 0"/>
+    <origin xyz="-0.22513 -0.1925 0.07335" rpy="1.57 1.0472 0"/>
     <axis   xyz="0 0 1"/>
-    <limit lower="0" upper="3.14" effort="1000" velocity="1"/>
+    <limit lower="0" upper="6.25" effort="1000" velocity="1"/>
   </joint>
   <!-- ──────────────── VIRTUAL JOINTS FOR SPEEDS ──────────────── -->
-  <!-- линейная скорость -->
-  <link name="lin_vel_link">
+  <link name="wheel_left_link">
     <inertial><mass value="1e-6"/><origin xyz="0 0 0" rpy="0 0 0"/>
       <inertia ixx="1e-6" iyy="1e-6" izz="1e-6" ixy="0" ixz="0" iyz="0"/>
     </inertial>
   </link>
-  <joint name="lin_vel_joint" type="continuous">
-    <parent link="base_link"/><child link="lin_vel_link"/>
-    <origin xyz="0 0 0" rpy="0 0 0"/><axis xyz="1 0 0"/>
+  <joint name="wheel_left_joint" type="continuous">
+    <parent link="base_link"/><child link="wheel_left_link"/>
+    <origin xyz="0 0.19 0.07335" rpy="0 0 0"/>
+    <axis   xyz="0 1 0"/>
   </joint>
-  <!-- угловая скорость -->
-  <link name="ang_vel_link">
+  <link name="wheel_right_link">
     <inertial><mass value="1e-6"/><origin xyz="0 0 0" rpy="0 0 0"/>
       <inertia ixx="1e-6" iyy="1e-6" izz="1e-6" ixy="0" ixz="0" iyz="0"/>
     </inertial>
   </link>
-  <joint name="ang_vel_joint" type="continuous">
-    <parent link="base_link"/><child link="ang_vel_link"/>
-    <origin xyz="0 0 0" rpy="0 0 0"/><axis xyz="0 0 1"/>
+  <joint name="wheel_right_joint" type="continuous">
+    <parent link="base_link"/><child link="wheel_right_link"/>
+    <origin xyz="0 -0.19 0.07335" rpy="0 0 0"/>
+    <axis   xyz="0 1 0"/>
   </joint>
 </robot>

Commit message: fixed lidar sim & controllers real description - returned to geom joint, bringup stable

File: src/tracked_description/config/t21.ros2_control.xacro (robot description, xacro)
@@ -7,30 +7,30 @@
   ================================================================= -->
   <xacro:unless value="$(arg use_sim_time)">
-    <xacro:macro name="t21_ros2_control" params="name prefix">
-      <ros2_control name="${name}_hw" type="system">
-        <!-- аппаратный плагин -->
-        <hardware>
-          <plugin>t21_hardware/T21TrackedHardware</plugin>
-          <!-- при необходимости можно добавить <param …/> -->
-        </hardware>
-        <!-- виртуальный сустав линейной скорости -->
-        <joint name="${prefix}wheel_left_joint">
-          <command_interface name="velocity"/>
-          <state_interface   name="velocity"/>
-          <state_interface name="position"/>
-        </joint>
-        <!-- виртуальный сустав угловой скорости -->
-        <joint name="${prefix}wheel_right_joint">
-          <command_interface name="velocity"/>
-          <state_interface   name="velocity"/>
-          <state_interface name="position"/>
-        </joint>
-        <!-- реальный сустав флиппера / стрелы -->
-        <joint name="${prefix}flipper_joint">
-          <command_interface name="position"/>
-          <state_interface   name="position"/>
-        </joint>
-      </ros2_control>
-    </xacro:macro>
+  <xacro:macro name="t21_ros2_control" params="name prefix">
+    <ros2_control name="${name}_hw" type="system">
+      <!-- аппаратный плагин -->
+      <hardware>
+        <plugin>t21_hardware/T21TrackedHardware</plugin>
+        <!-- при необходимости можно добавить <param …/> -->
+      </hardware>
+      <!-- виртуальный сустав линейной скорости -->
+      <joint name="${prefix}wheel_left_joint">
+        <command_interface name="velocity"/>
+        <state_interface   name="velocity"/>
+        <state_interface name="position"/>
+      </joint>
+      <!-- виртуальный сустав угловой скорости -->
+      <joint name="${prefix}wheel_right_joint">
+        <command_interface name="velocity"/>
+        <state_interface   name="velocity"/>
+        <state_interface name="position"/>
+      </joint>
+      <!-- реальный сустав флиппера / стрелы -->
+      <joint name="${prefix}geom_joint">
+        <command_interface name="position"/>
+        <state_interface   name="position"/>
+      </joint>
+    </ros2_control>
+  </xacro:macro>
     <!-- Вызываем макрос, передавая имя и префикс -->
     <xacro:t21_ros2_control name="t21" prefix="$(arg prefix)"/>

File: src/tracked_description/urdf/lidar.xacro (robot description, xacro)
@@ -25,11 +25,11 @@
       lasers="16"
       samples="400"
-      min_range="0.5"
+      collision_range="0.3"
+      min_range="0.1"
       max_range="25.0"
+      noise="0.0"
+      min_angle="-${pi/2}"
+      max_angle="${pi/2}"
       gpu="false">
-      <!--
-      min_angle="-0.0"
-      max_angle="6.2831853"
-      -->
       <origin xyz="0 0 -0.035" rpy="0 0 0" />
     </xacro:VLP-16>

File: src/tracked_description/urdf/tracked_robot.urdf.xacro (robot description, xacro)
@@ -35,5 +35,5 @@
                    xyz="0 0 0"/>
   <!-- ──────────────── FLIPPER / GEOMETRY ──────────────── -->
-  <xacro:add_link  name="flipperlink"
+  <xacro:add_link  name="geom_link"
                    mesh="fliper.stl"
                    scale="${scale_small}"
@@ -41,7 +41,7 @@
                    rpy="0 0 0"
                    xyz="0 0 0"/>
-  <joint name="flipper_joint" type="revolute">
+  <joint name="geom_joint" type="revolute">
     <parent link="base_link"/>
-    <child  link="flipper_link"/>
+    <child  link="geom_link"/>
     <origin xyz="0.22513 0.1925 0.07335" rpy="-1.57 4.71239 0"/>
     <axis   xyz="0 0 1"/>
